File: LCD1888BoardDriver/LCD1888BoardDriver.kicad_pcb (KiCad board)
At the start: 2 copper layers, 38.3 x 76.5 mm, 20 parts, among them J1 Conn_01x05_Male, J2 Conn_01x02_Male, J3 Conn_01x02_Male, U1 HT1621B, U2 DE113-XX-XX, Y1 32768

Commit message: Add files via upload
Parts:
- added H10: MountingHole_Pad, MountingHole:MountingHole_3.2mm_M3_Pad_Via, F.Cu at (113.7, 51.6)
- added H11: MountingHole_Pad, MountingHole:MountingHole_3.2mm_M3_Pad_Via, F.Cu at (113.7, 96.9)
- added H12: MountingHole, Symbol:KiCad-Logo2_5mm_SilkScreen, F.Cu at (113.7, 76.2)
- added H13: MountingHole, Symbol:OSHW-Logo2_7.3x6mm_SilkScreen, F.Cu at (161.0, 74.9)
- added H14: MountingHole, Symbol:Symbol_CC-ShareAlike_SilkscreenTop_Small, F.Cu at (161.3, 83.7)
- added H15: MountingHole, Symbol:WEEE-Logo_4.2x6mm_SilkScreen, F.Cu at (144.7, 104.7)
- added H16: MountingHole, Symbol:WEEE-Logo_4.2x6mm_SilkScreen, F.Cu at (161.2, 65.5)
- added H8: MountingHole_Pad, MountingHole:MountingHole_3.2mm_M3_Pad_Via, F.Cu at (161.3, 96.8)
- added H9: MountingHole_Pad, MountingHole:MountingHole_3.2mm_M3_Pad_Via, F.Cu at (161.2, 51.5)
- J1: value Conn_01x05_Male -> Data & Power 5V; footprint Connector_JST:JST_XH_S5B-XH-A_1x05_P2.50mm_Horizontal -> Connector_JST:JST_XH_S6B-XH-A-1_1x06_P2.50mm_Horizontal
- J2: value Conn_01x02_Male -> Interrupt OUT
- J3: value Conn_01x02_Male -> Power 5V
- moved H7 4.53 mm to (134.4, 104.3)
- moved J1 2.28 mm to (126.4, 91.4)
- moved H2 2.21 mm to (121.9, 104.6)
- moved H3 2.21 mm to (153.1, 104.6)
- moved H1 2.13 mm to (121.9, 43.5)
- moved H4 2.13 mm to (153.0, 43.5)
- moved H5 1.83 mm to (137.8, 43.3)
Connections:
- J3 pad 2: Net-(L1-Pad2) -> Net-(J3-Pad2)
- L1 pad 2: Net-(L1-Pad2) -> Net-(J3-Pad2)
Routing:
- net GND: track 223.6 -> 0.00 mm, vias 0 -> 6
- net Net-(J2-Pad2): track 77.2 -> 23.6 mm, vias 0 -> 1
- net Net-(U1-Pad12): track 15.6 -> 36.3 mm
- net Net-(U1-Pad23): track 34.4 -> 55.0 mm, vias 1 -> 0
- net Net-(RV1-Pad1): track 28.2 -> 48.1 mm
- net Net-(J3-Pad2): track 0.00 -> 18.7 mm
- net Net-(U1-Pad11): track 28.0 -> 46.7 mm, vias 0 -> 1
- net Net-(C1-Pad1): track 66.7 -> 78.9 mm, vias 0 -> 2
- net Net-(L1-Pad2): track 8.88 -> 0.00 mm
- net Net-(U1-Pad5): track 23.2 -> 30.6 mm
- net Net-(U1-Pad15): track 31.6 -> 38.3 mm
- net Net-(U1-Pad19): track 40.6 -> 47.3 mm, vias 1 -> 0
- net Net-(U1-Pad32): track 27.5 -> 21.3 mm
- net Net-(U1-Pad4): track 22.5 -> 28.5 mm
- net Net-(U1-Pad42): track 24.6 -> 18.7 mm
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- added copper zone on B.Cu, net GND
- added copper zone on F.Cu, net GND
Other:
- board size 38.3 x 76.5 mm -> 54.5 x 68.2 mm
- board text added: "SaLe fecit 2022"
- board text added: "https://github.com/SaLeeC/ LCD1888-Board-Driver"
- board text added: "https://github.com/SaLeeC/LCD1888-Board-Driver"
